File: PCB/CapacitiveLedFadeTiny/CapacitiveLedFadeTiny.kicad_sch (KiCad schematic)
At the start: 7 parts, among them J1 Bus In, J2 Bus Out, J3 LEDs, J4 Antenna, U1 ATTINY85-20SU

Commit message: Update board layout
the attiny is actually a wider footprint :kms:
this is why we do prototype boards
Parts:
- U1: footprint digikey-footprints:SOIC-8_W5.3mm -> Package_SO:SOIC-8_5.23x5.23mm_P1.27mm
Changed lines of the file:
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@@
       (effects (font (size 1.524 1.524)) (justify left))
     )
-    (property "Footprint" "digikey-footprints:SOIC-8_W5.3mm" (at 155.575 56.515 0)
+    (property "Footprint" "Package_SO:SOIC-8_5.23x5.23mm_P1.27mm" (at 155.575 56.515 0)
       (effects (font (size 1.524 1.524)) (justify left) hide)
     )

Commit message: v2 of I2C board
Parts:
- added J6: Power Inject, Library:SCREW_TERMINAL_5mm_01x02, symbol Connector:Screw_Terminal_01x02
- added Pad1: 1, Library:TestPoint_Pad_1.5mm_circular, symbol Connector_Generic:Conn_01x01
- added Pad2: 2, Library:TestPoint_Pad_1.5mm_circular, symbol Connector_Generic:Conn_01x01
- added Pad3: 3, Library:TestPoint_Pad_1.5mm_circular, symbol Connector_Generic:Conn_01x01
- added Pad6: 6, Library:TestPoint_Pad_1.5mm_circular, symbol Connector_Generic:Conn_01x01
- added PadGnd1: GND, Library:TestPoint_Pad_1.5mm_circular, symbol Connector_Generic:Conn_01x01
- added PadSclk1: SCLK, Library:TestPoint_Pad_1.5mm_circular, symbol Connector_Generic:Conn_01x01
- added PadSda1: SDA, Library:TestPoint_Pad_1.5mm_circular, symbol Connector_Generic:Conn_01x01
- added PadVCC1: VCC, Library:TestPoint_Pad_1.5mm_circular, symbol Connector_Generic:Conn_01x01
- ATTiny85: renamed from U1; footprint Package_SO:SOIC-8_5.23x5.23mm_P1.27mm -> ATTINY85-20SFR:SOIC127P798X216-8N
- BusIn1: renamed from J1; footprint Connector_PinHeader_2.54mm:PinHeader_1x04_P2.54mm_Vertical -> Connector_JST:JST_XH_B4B-XH-A_1x04_P2.50mm_Vertical
- BusOut1: renamed from J2; footprint Connector_PinHeader_2.54mm:PinHeader_1x04_P2.54mm_Vertical -> Connector_JST:JST_XH_B4B-XH-A_1x04_P2.50mm_Vertical
- LED3: renamed from J3; footprint Connector_PinHeader_2.54mm:PinHeader_1x03_P2.54mm_Vertical -> Connector_JST:JST_XH_B3B-XH-A_1x03_P2.50mm_Vertical
Connections:
- net GND: now also J6.2 (Pin_2), PadGnd1.1 (Pin_1)
- net SCLK: now also PadSclk1.1 (Pin_1)
- net SDA: now also PadSda1.1 (Pin_1)
- net VCC: now also J6.1 (Pin_1), PadVCC1.1 (Pin_1)
- net 6: now reaches ATTiny85.6 (PB1), LED3.2 (Pin_2)
- net 6: now also Pad6.1 (Pin_1)
- net 1: now reaches ATTiny85.1 (PB5)
- net 1: now also Pad1.1 (Pin_1)
- net 2: now reaches ATTiny85.2 (PB3), J4.1 (Pin_1)
- net 2: now also Pad2.1 (Pin_1)
- net 3: now reaches ATTiny85.3 (PB4)
- net 3: now also Pad3.1 (Pin_1)
- no-connect marks 2 -> 0
Other:
- note added: "Pogo Pin Programming Points"
