File: PCB/CapacitiveLedFadeTiny/CapacitiveLedFadeTiny.kicad_sch (KiCad schematic)
At the start: 17 parts, among them J1 Antenna, J3 PadUPDI, J4 PadTX, J5 PadRX, J6 Power Inject, U1 ATtiny3224-X

Commit message: pcb v3.1
Parts:
- J1: footprint TestPoint:TestPoint_Pad_1.0x1.0mm -> CapacitiveLedFadeLibrary:CapacitiveAntenna
Connections:
- net SCLK: now also BusIn1.3 (Pin_3), BusOut1.3 (Pin_3); no longer BusIn1.4 (Pin_4), BusOut1.4 (Pin_4)
- net SDA: now also BusIn1.4 (Pin_4), BusOut1.4 (Pin_4); no longer BusIn1.3 (Pin_3), BusOut1.3 (Pin_3)
Other:
- moved on the sheet: BusIn1, BusOut1
Changed lines of the file:
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@@
   (no_connect (at 169.545 111.125))
   (no_connect (at 184.15 102.235))
-  (wire (pts (xy 130.81 40.005) (xy 117.475 40.005))
-    (stroke (width 0) (type default))
-  )
   (wire (pts (xy 82.55 35.56) (xy 92.075 35.56))
     (stroke (width 0) (type default))
   )
-  (wire (pts (xy 117.475 40.005) (xy 117.475 39.37))
-    (stroke (width 0) (type default))
-  )
-  (wire (pts (xy 117.475 42.545) (xy 117.475 45.085))
-    (stroke (width 0) (type default))
-  )
   (wire (pts (xy 179.705 87.63) (xy 179.705 99.695))
     (stroke (width 0) (type default))
@@
     (stroke (width 0) (type default))
   )
-  (wire (pts (xy 130.175 36.195) (xy 130.175 37.465))
-    (stroke (width 0) (type default))
-  )
-  (wire (pts (xy 95.885 43.18) (xy 95.885 48.895))
+  (wire (pts (xy 95.25 43.18) (xy 95.25 48.26))
+    (stroke (width 0) (type default))
+  )
+  (wire (pts (xy 130.175 36.195) (xy 130.175 38.1))
+    (stroke (width 0) (type default))
+  )
+  (wire (pts (xy 129.54 34.925) (xy 125.73 34.925))
     (stroke (width 0) (type default))
   )
@@
     (stroke (width 0) (type default))
   )
-  (wire (pts (xy 125.73 34.925) (xy 130.81 34.925))
+  (wire (pts (xy 129.54 35.56) (xy 130.81 35.56))
     (stroke (width 0) (type default))
   )
@@
     (stroke (width 0) (type default))
   )
-  (wire (pts (xy 86.995 43.815) (xy 93.98 43.815))
-    (stroke (width 0) (type default))
-  )
-  (wire (pts (xy 130.81 42.545) (xy 117.475 42.545))
-    (stroke (width 0) (type default))
-  )
-  (wire (pts (xy 82.55 38.1) (xy 95.885 38.1))
+  (wire (pts (xy 82.55 38.1) (xy 95.25 38.1))
+    (stroke (width 0) (type default))
+  )
+  (wire (pts (xy 125.73 40.64) (xy 125.73 49.53))
     (stroke (width 0) (type default))
   )
@@
     (stroke (width 0) (type default))
   )
+  (wire (pts (xy 129.54 35.56) (xy 129.54 34.925))
+    (stroke (width 0) (type default))
+  )
   (wire (pts (xy 181.61 92.075) (xy 181.61 97.155))
     (stroke (width 0) (type default))
@@
     (stroke (width 0) (type default))
   )
-  (wire (pts (xy 95.25 40.64) (xy 95.885 40.64))
-    (stroke (width 0) (type default))
-  )
   (wire (pts (xy 179.705 99.695) (xy 184.15 99.695))
     (stroke (width 0) (type default))
   )
+  (wire (pts (xy 95.25 40.64) (xy 86.36 40.64))
+    (stroke (width 0) (type default))
+  )
   (wire (pts (xy 179.07 74.93) (xy 179.07 85.09))
     (stroke (width 0) (type default))
   )
-  (wire (pts (xy 95.25 41.91) (xy 95.25 40.64))
+  (wire (pts (xy 130.81 40.64) (xy 125.73 40.64))
     (stroke (width 0) (type default))
   )
@@
     (stroke (width 0) (type default))
   )
+  (wire (pts (xy 130.81 43.18) (xy 130.81 49.53))
+    (stroke (width 0) (type default))
+  )
   (wire (pts (xy 181.61 97.155) (xy 184.15 97.155))
     (stroke (width 0) (type default))
@@
     (stroke (width 0) (type default))
   )
-  (wire (pts (xy 130.175 37.465) (xy 130.81 37.465))
+  (wire (pts (xy 130.175 38.1) (xy 130.81 38.1))
     (stroke (width 0) (type default))
   )
@@
     (stroke (width 0) (type default))
   )
+  (wire (pts (xy 86.36 40.64) (xy 86.36 53.34))
+    (stroke (width 0) (type default))
+  )
   (wire (pts (xy 149.86 57.785) (xy 149.86 62.23))
     (stroke (width 0) (type default))
@@
     (stroke (width 0) (type default))
   )
-  (wire (pts (xy 92.075 35.56) (xy 95.885 35.56))
+  (wire (pts (xy 92.075 35.56) (xy 95.25 35.56))
     (stroke (width 0) (type default))
   )
@@
     (stroke (width 0) (type default))
   )
-  (wire (pts (xy 93.98 41.91) (xy 93.98 43.815))
-    (stroke (width 0) (type default))
-  )
-  (wire (pts (xy 93.98 41.91) (xy 95.25 41.91))
-    (stroke (width 0) (type default))
-  )
   (wire (pts (xy 113.665 36.195) (xy 130.175 36.195))
     (stroke (width 0) (type default))
   )
+  (wire (pts (xy 130.81 49.53) (xy 132.08 49.53))
+    (stroke (width 0) (type default))
+  )
   (wire (pts (xy 169.545 80.01) (xy 169.545 106.045))
     (stroke (width 0) (type default))
@@
     (effects (font (size 1.27 1.27)) (justify left bottom))
   )
+  (label "SCLK" (at 125.73 49.53 0) (fields_autoplaced)
+    (effects (font (size 1.27 1.27)) (justify left bottom))
+  )
   (label "UPDI" (at 86.995 78.74 0) (fields_autoplaced)
     (effects (font (size 1.27 1.27)) (justify left bottom))
   )
+  (label "SDA" (at 95.25 48.26 0) (fields_autoplaced)
+    (effects (font (size 1.27 1.27)) (justify left bottom))
+  )
   (label "RX" (at 88.9 95.25 0) (fields_autoplaced)
     (effects (font (size 1.27 1.27)) (justify left bottom))
@@
     (effects (font (size 1.27 1.27)) (justify left bottom))
   )
-  (label "SDA" (at 117.475 39.37 0) (fields_autoplaced)
-    (effects (font (size 1.27 1.27)) (justify left bottom))
-  )
   (label "LED_Signal" (at 181.61 92.075 0) (fields_autoplaced)
     (effects (font (size 1.27 1.27)) (justify left bottom))
@@
     (effects (font (size 1.27 1.27)) (justify left bottom))
   )
-  (label "SCLK" (at 117.475 45.085 0) (fields_autoplaced)
-    (effects (font (size 1.27 1.27)) (justify left bottom))
-  )
   (label "LED_Signal" (at 209.55 86.995 0) (fields_autoplaced)
     (effects (font (size 1.27 1.27)) (justify left bottom))
@@
     (effects (font (size 1.27 1.27)) (justify left bottom))
   )
-  (label "SDA" (at 86.995 43.815 0) (fields_autoplaced)
-    (effects (font (size 1.27 1.27)) (justify left bottom))
-  )
   (label "SDA" (at 103.505 71.755 0) (fields_autoplaced)
     (effects (font (size 1.27 1.27)) (justify left bottom))
@@
     (effects (font (size 1.27 1.27)) (justify left bottom))
   )
-  (label "SCLK" (at 95.885 48.895 0) (fields_autoplaced)
+  (label "SDA" (at 132.08 49.53 0) (fields_autoplaced)
+    (effects (font (size 1.27 1.27)) (justify left bottom))
+  )
+  (label "SCLK" (at 86.36 53.34 0) (fields_autoplaced)
     (effects (font (size 1.27 1.27)) (justify left bottom))
   )
@@
       (effects (font (size 1.27 1.27)))
     )
-    (property "Footprint" "TestPoint:TestPoint_Pad_1.0x1.0mm" (at 207.645 74.93 0)
+    (property "Footprint" "CapacitiveLedFadeLibrary:CapacitiveAntenna" (at 207.645 74.93 0)
       (effects (font (size 1.27 1.27)) hide)
     )
@@
     )
   )
-  (symbol (lib_id "Connector_Generic:Conn_01x04") (at 135.89 37.465 0) (unit 1)
-    (in_bom yes) (on_board yes) (dnp no) (fields_autoplaced)
-    (property "Reference" "BusOut1" (at 138.43 37.465 0)
-      (effects (font (size 1.27 1.27)) (justify left))
-    )
-    (property "Value" "Bus Out" (at 138.43 40.005 0)
+  (symbol (lib_id "Connector_Generic:Conn_01x04") (at 135.89 38.1 0) (unit 1)
+    (in_bom yes) (on_board yes) (dnp no) (fields_autoplaced)
+    (property "Reference" "BusOut1" (at 138.43 38.1 0)
+      (effects (font (size 1.27 1.27)) (justify left))
+    )
+    (property "Value" "Bus Out" (at 138.43 40.64 0)
       (effects (font (size 1.27 1.27)) (justify left) hide)
     )
-    (property "Footprint" "Connector_JST:JST_SH_BM04B-SRSS-TB_1x04-1MP_P1.00mm_Vertical" (at 135.89 37.465 0)
-      (effects (font (size 1.27 1.27)) hide)
-    )
-    (property "Datasheet" "~" (at 135.89 37.465 0)
+    (property "Footprint" "Connector_JST:JST_SH_BM04B-SRSS-TB_1x04-1MP_P1.00mm_Vertical" (at 135.89 38.1 0)
+      (effects (font (size 1.27 1.27)) hide)
+    )
+    (property "Datasheet" "~" (at 135.89 38.1 0)
       (effects (font (size 1.27 1.27)) hide)
     )
@@
     )
   )
-  (symbol (lib_id "Connector_Generic:Conn_01x04") (at 100.965 38.1 0) (unit 1)
-    (in_bom yes) (on_board yes) (dnp no) (fields_autoplaced)
-    (property "Reference" "BusIn1" (at 104.14 38.1 0)
-      (effects (font (size 1.27 1.27)) (justify left))
-    )
-    (property "Value" "Bus In" (at 104.14 40.64 0)
+  (symbol (lib_id "Connector_Generic:Conn_01x04") (at 100.33 38.1 0) (unit 1)
+    (in_bom yes) (on_board yes) (dnp no) (fields_autoplaced)
+    (property "Reference" "BusIn1" (at 103.505 38.1 0)
+      (effects (font (size 1.27 1.27)) (justify left))
+    )
+    (property "Value" "Bus In" (at 103.505 40.64 0)
       (effects (font (size 1.27 1.27)) (justify left) hide)
     )
-    (property "Footprint" "Connector_JST:JST_SH_BM04B-SRSS-TB_1x04-1MP_P1.00mm_Vertical" (at 100.965 38.1 0)
-      (effects (font (size 1.27 1.27)) hide)
-    )
-    (property "Datasheet" "~" (at 100.965 38.1 0)
-      (effects (font (size 1.27 1.27)) hide)
-    )
+    (property "Footprint" "Connector_JST:JST_SH_BM04B-SRSS-TB_1x04-1MP_P1.00mm_Vertical" (at 100.33 38.1 0)
+      (effects (font (size 1.27 1.27)) hide)
+    )
+    (property "Datasheet" "~" (at 100.33 38.1 0)
+      (effects (font (size 1.27 1.27)) hide)
+    )

Commit message: v3.2 pcb, changed to PA connectors
Parts:
- BusIn1, BusOut1: footprint Connector_JST:JST_SH_BM04B-SRSS-TB_1x04-1MP_P1.00mm_Vertical -> digikey-footprints:CONN_BM04B-PASS-1-TFTLFSN_JST
- LED_EXT1: footprint Connector_JST:JST_SH_BM03B-SRSS-TB_1x03-1MP_P1.00mm_Vertical -> digikey-footprints:BM03B-PASS-1-TFT
Changed lines of the file:
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@@
       (effects (font (size 1.27 1.27)) (justify left) hide)
     )
-    (property "Footprint" "Connector_JST:JST_SH_BM04B-SRSS-TB_1x04-1MP_P1.00mm_Vertical" (at 135.89 38.1 0)
+    (property "Footprint" "digikey-footprints:CONN_BM04B-PASS-1-TFTLFSN_JST" (at 135.89 38.1 0)
       (effects (font (size 1.27 1.27)) hide)
     )
@@
       (effects (font (size 1.27 1.27)) (justify left) hide)
     )
-    (property "Footprint" "Connector_JST:JST_SH_BM03B-SRSS-TB_1x03-1MP_P1.00mm_Vertical" (at 209.55 102.235 0)
+    (property "Footprint" "digikey-footprints:BM03B-PASS-1-TFT" (at 209.55 102.235 0)
       (effects (font (size 1.27 1.27)) hide)
     )
@@
       (effects (font (size 1.27 1.27)) (justify left) hide)
     )
-    (property "Footprint" "Connector_JST:JST_SH_BM04B-SRSS-TB_1x04-1MP_P1.00mm_Vertical" (at 100.33 38.1 0)
-      (effects (font (size 1.27 1.27)) hide)
-    )
+    (property "Footprint" "digikey-footprints:CONN_BM04B-PASS-1-TFTLFSN_JST" (at 100.33 38.1 0)
+      (effects (font (size 1.27 1.27)) hide)
+    )
