File: PCB/CapacitiveLedFadeTiny/_autosave-CapacitiveLedFadeTiny.kicad_sch (KiCad schematic)
At the start: 17 parts, among them J1 Antenna, J3 PadUPDI, J4 PadTX, J5 PadRX, J6 Power Inject, U1 ATtiny3224-X

Commit message: v3 pcb
Parts:
- J1: footprint TestPoint:TestPoint_Pad_1.0x1.0mm -> CapacitiveLedFadeLibrary:CapacitiveAntenna
Changed lines of the file:
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@@
       (effects (font (size 1.27 1.27)))
     )
-    (property "Footprint" "TestPoint:TestPoint_Pad_1.0x1.0mm" (at 207.645 74.93 0)
+    (property "Footprint" "CapacitiveLedFadeLibrary:CapacitiveAntenna" (at 207.645 74.93 0)
       (effects (font (size 1.27 1.27)) hide)
     )
